Commit message: quelques ajustement pour pouvoir utilisé urdf arm

File: reachy.urdf (robot description, URDF)
Before this commit: robot reachy2, 78 links, 77 joints
Links:
- link base_link: geometry collision cylinder length=0.2609 radius=0.245; visual mesh filename=file:////home/kloe-bonnet/Documents/ENSEIRB/essai/projet_po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
- link head: geometry collision mesh filename=file:///home/kloe-bonnet/Documents/ENSEIRB/essai/projet_pol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; visual mesh filename=file:///home/kloe-bonnet/Documents/ENSEIRB/essai/projet_pol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
- link l_elbow_arm_link: geometry collision mesh filename=file:///home/kloe-bonnet/Documents/ENSEIRB/essai/projet_pol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; visual mesh filename=file:///home/kloe-bonnet/Documents/ENSEIRB/essai/projet_pol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
- link l_elbow_first_link: geometry visual mesh filename=file:///home/kloe-bonnet/Documents/ENSEIRB/essai/projet_pol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
- link l_elbow_forearm_link: geometry collision mesh filename=file:///home/kloe-bonnet/Documents/ENSEIRB/essai/projet_pol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; visual mesh filename=file:///home/kloe-bonnet/Documents/ENSEIRB/essai/projet_pol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
- link l_hand_distal_link: geometry collision mesh filename=file:///home/kloe-bonnet/Documents/ENSEIRB/essai/projet_pol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; visual mesh filename=file:///home/kloe-bonnet/Documents/ENSEIRB/essai/projet_pol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
- link l_hand_distal_mimic_link: geometry collision mesh filename=file:///home/kloe-bonnet/Documents/ENSEIRB/essai/projet_pol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; visual mesh filename=file:///home/kloe-bonnet/Documents/ENSEIRB/essai/projet_pol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
- link l_hand_palm_link: geometry collision mesh filename=file:///home/kloe-bonnet/Documents/ENSEIRB/essai/projet_pol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; visual mesh filename=file:///home/kloe-bonnet/Documents/ENSEIRB/essai/projet_pol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
- link l_hand_proximal_link: geometry collision mesh filename=file:///home/kloe-bonnet/Documents/ENSEIRB/essai/projet_pol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; visual mesh filename=file:///home/kloe-bonnet/Documents/ENSEIRB/essai/projet_pol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
- link l_hand_proximal_mimic_link: geometry collision mesh filename=file:///home/kloe-bonnet/Documents/ENSEIRB/essai/projet_pol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; visual mesh filename=file:///home/kloe-bonnet/Documents/ENSEIRB/essai/projet_pol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
- link l_shoulder_first_link: geometry visual mesh filename=file:///home/kloe-bonnet/Documents/ENSEIRB/essai/projet_pol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
- link r_elbow_arm_link: geometry collision mesh filename=file:///home/kloe-bonnet/Documents/ENSEIRB/essai/projet_pol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; visual mesh filename=file:///home/kloe-bonnet/Documents/ENSEIRB/essai/projet_pol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
- link r_elbow_first_link: geometry visual mesh filename=file:///home/kloe-bonnet/Documents/ENSEIRB/essai/projet_pol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
- link r_elbow_forearm_link: geometry collision mesh filename=file:///home/kloe-bonnet/Documents/ENSEIRB/essai/projet_pol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; visual mesh filename=file:///home/kloe-bonnet/Documents/ENSEIRB/essai/projet_pol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
- link r_hand_distal_link: geometry collision mesh filename=file:///home/kloe-bonnet/Documents/ENSEIRB/essai/projet_pol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; visual mesh filename=file:///home/kloe-bonnet/Documents/ENSEIRB/essai/projet_pol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
- link r_hand_distal_mimic_link: geometry collision mesh filename=file:///home/kloe-bonnet/Documents/ENSEIRB/essai/projet_pol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; visual mesh filename=file:///home/kloe-bonnet/Documents/ENSEIRB/essai/projet_pol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
- link r_hand_palm_link: geometry collision mesh filename=file:///home/kloe-bonnet/Documents/ENSEIRB/essai/projet_pol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; visual mesh filename=file:///home/kloe-bonnet/Documents/ENSEIRB/essai/projet_pol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
- link r_hand_proximal_link: geometry collision mesh filename=file:///home/kloe-bonnet/Documents/ENSEIRB/essai/projet_pol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; visual mesh filename=file:///home/kloe-bonnet/Documents/ENSEIRB/essai/projet_pol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
- link r_hand_proximal_mimic_link: geometry collision mesh filename=file:///home/kloe-bonnet/Documents/ENSEIRB/essai/projet_pol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; visual mesh filename=file:///home/kloe-bonnet/Documents/ENSEIRB/essai/projet_pol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
- link r_shoulder_first_link: geometry visual mesh filename=file:///home/kloe-bonnet/Documents/ENSEIRB/essai/projet_pol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
- link torso: geometry collision mesh filename=file:///home/kloe-bonnet/Documents/ENSEIRB/essai/projet_pol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; visual mesh filename=file:///home/kloe-bonnet/Documents/ENSEIRB/essai/projet_pol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

Commit message: avancement fonction mais problemes calcule cinematique directe, tests sauvegarde avant reunion securite

File: reachy.urdf (robot description, URDF)
Before this commit: robot reachy2, 78 links, 77 joints
Links:
- link base_link: geometry collision cylinder length=0.2609 radius=0.245; visual mesh filename=file:////home/kloe-bonnet/Documents/ENSEIRB/dfdf/projet_pol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
- link head: geometry collision mesh filename=file:///home/kloe-bonnet/Documents/ENSEIRB/dfdf/projet_poll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; visual mesh filename=file:///home/kloe-bonnet/Documents/ENSEIRB/dfdf/projet_poll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
- link l_elbow_arm_link: geometry collision mesh filename=file:///home/kloe-bonnet/Documents/ENSEIRB/dfdf/projet_poll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; visual mesh filename=file:///home/kloe-bonnet/Documents/ENSEIRB/dfdf/projet_poll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
- link l_elbow_first_link: geometry visual mesh filename=file:///home/kloe-bonnet/Documents/ENSEIRB/dfdf/projet_poll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
- link l_elbow_forearm_link: geometry collision mesh filename=file:///home/kloe-bonnet/Documents/ENSEIRB/dfdf/projet_poll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; visual mesh filename=file:///home/kloe-bonnet/Documents/ENSEIRB/dfdf/projet_poll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
- link l_hand_distal_link: geometry collision mesh filename=file:///home/kloe-bonnet/Documents/ENSEIRB/dfdf/projet_poll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; visual mesh filename=file:///home/kloe-bonnet/Documents/ENSEIRB/dfdf/projet_poll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
- link l_hand_distal_mimic_link: geometry collision mesh filename=file:///home/kloe-bonnet/Documents/ENSEIRB/dfdf/projet_poll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; visual mesh filename=file:///home/kloe-bonnet/Documents/ENSEIRB/dfdf/projet_poll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
- link l_hand_palm_link: geometry collision mesh filename=file:///home/kloe-bonnet/Documents/ENSEIRB/dfdf/projet_poll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; visual mesh filename=file:///home/kloe-bonnet/Documents/ENSEIRB/dfdf/projet_poll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
- link l_hand_proximal_link: geometry collision mesh filename=file:///home/kloe-bonnet/Documents/ENSEIRB/dfdf/projet_poll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; visual mesh filename=file:///home/kloe-bonnet/Documents/ENSEIRB/dfdf/projet_poll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
- link l_hand_proximal_mimic_link: geometry collision mesh filename=file:///home/kloe-bonnet/Documents/ENSEIRB/dfdf/projet_poll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; visual mesh filename=file:///home/kloe-bonnet/Documents/ENSEIRB/dfdf/projet_poll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
- link l_shoulder_first_link: geometry visual mesh filename=file:///home/kloe-bonnet/Documents/ENSEIRB/dfdf/projet_poll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
- link r_elbow_arm_link: geometry collision mesh filename=file:///home/kloe-bonnet/Documents/ENSEIRB/dfdf/projet_poll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; visual mesh filename=file:///home/kloe-bonnet/Documents/ENSEIRB/dfdf/projet_poll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
- link r_elbow_first_link: geometry visual mesh filename=file:///home/kloe-bonnet/Documents/ENSEIRB/dfdf/projet_poll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
- link r_elbow_forearm_link: geometry collision mesh filename=file:///home/kloe-bonnet/Documents/ENSEIRB/dfdf/projet_poll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; visual mesh filename=file:///home/kloe-bonnet/Documents/ENSEIRB/dfdf/projet_poll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
- link r_hand_distal_link: geometry collision mesh filename=file:///home/kloe-bonnet/Documents/ENSEIRB/dfdf/projet_poll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; visual mesh filename=file:///home/kloe-bonnet/Documents/ENSEIRB/dfdf/projet_poll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
- link r_hand_distal_mimic_link: geometry collision mesh filename=file:///home/kloe-bonnet/Documents/ENSEIRB/dfdf/projet_poll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; visual mesh filename=file:///home/kloe-bonnet/Documents/ENSEIRB/dfdf/projet_poll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
- link r_hand_palm_link: geometry collision mesh filename=file:///home/kloe-bonnet/Documents/ENSEIRB/dfdf/projet_poll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; visual mesh filename=file:///home/kloe-bonnet/Documents/ENSEIRB/dfdf/projet_poll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
- link r_hand_proximal_link: geometry collision mesh filename=file:///home/kloe-bonnet/Documents/ENSEIRB/dfdf/projet_poll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; visual mesh filename=file:///home/kloe-bonnet/Documents/ENSEIRB/dfdf/projet_poll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
- link r_hand_proximal_mimic_link: geometry collision mesh filename=file:///home/kloe-bonnet/Documents/ENSEIRB/dfdf/projet_poll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; visual mesh filename=file:///home/kloe-bonnet/Documents/ENSEIRB/dfdf/projet_poll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
- link r_shoulder_first_link: geometry visual mesh filename=file:///home/kloe-bonnet/Documents/ENSEIRB/dfdf/projet_poll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
- link torso: geometry collision mesh filename=file:///home/kloe-bonnet/Documents/ENSEIRB/dfdf/projet_poll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; visual mesh filename=file:///home/kloe-bonnet/Documents/ENSEIRB/dfdf/projet_poll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
